Commit message: Camera added to xacro file.

File: src/bioloid_typea_description/gazebo.xacro (robot description, xacro)
@@ -16,14 +16,53 @@
 		    <visualize>true</visualize>
 		</plugin>
-            <plugin name="p3d_base_controller" filename="libgazebo_ros_p3d.so">
-              <alwaysOn>true</alwaysOn>
-              <updateRate>50.0</updateRate>
-              <bodyName>base_link</bodyName>
-              <topicName>position</topicName>
-              <gaussianNoise>0.01</gaussianNoise>
-              <frameName>world</frameName>
-              <xyzOffsets>0 0 0</xyzOffsets>
-              <rpyOffsets>0 0 0</rpyOffsets>
+        <plugin name="p3d_base_controller" filename="libgazebo_ros_p3d.so">
+            <alwaysOn>true</alwaysOn>
+            <updateRate>50.0</updateRate>
+            <bodyName>base_link</bodyName>
+            <topicName>position</topicName>
+            <gaussianNoise>0.01</gaussianNoise>
+            <frameName>world</frameName>
+            <xyzOffsets>0 0 0</xyzOffsets>
+            <rpyOffsets>0 0 0</rpyOffsets>
+        </plugin>
+    </gazebo>
+    <gazebo reference="camera_link">
+        <sensor type="camera" name="camera">
+            <update_rate>30.0</update_rate>
+            <camera name="head">
+                <horizontal_fov>1.3962634</horizontal_fov>
+                <image>
+                  <width>800</width>
+                  <height>800</height>
+                  <format>R8G8B8</format>
+                </image>
+                <clip>
+                  <near>0.02</near>
+                  <far>300</far>
+                </clip>
+                <noise>
+                  <type>gaussian</type>
+                  <!-- Noise is sampled independently per pixel on each frame.
+                       That pixel's noise value is added to each of its color
+                       channels, which at that point lie in the range [0,1]. -->
+                  <mean>0.0</mean>
+                  <stddev>0.007</stddev>
+                </noise>
+            </camera>
+            <plugin name="camera_controller" filename="libgazebo_ros_camera.so">
+                <alwaysOn>true</alwaysOn>
+                <updateRate>0.0</updateRate>
+                <cameraName>camera</cameraName>
+                <imageTopicName>image_raw</imageTopicName>
+                <cameraInfoTopicName>camera_info</cameraInfoTopicName>
+                <frameName>camera_link</frameName>
+                <hackBaseline>0.07</hackBaseline>
+                <distortionK1>0.0</distortionK1>
+                <distortionK2>0.0</distortionK2>
+                <distortionK3>0.0</distortionK3>
+                <distortionT1>0.0</distortionT1>
+                <distortionT2>0.0</distortionT2>
             </plugin>
+        </sensor>
     </gazebo>
     <xacro:macro name="shoulder_swing_joint_gazebo" params="prefix">

File: src/bioloid_typea_description/typea.xacro (robot description, xacro)
@@ -35,5 +35,5 @@
     <xacro:include filename="$(find bioloid_typea_description)/std_parts.xacro"/>
      <xacro:property name="camera_link" value="0.01" />
-     <xacro:property name="height_camera" value="0.2"/>
+     <xacro:property name="height_camera" value="0.157"/>
      <xacro:property name="axel_offset" value="0.05"/>
     <!-- Camera -->
@@ -54,7 +54,7 @@
             <origin xyz="0 0 0" rpy="0 0 0"/>
             <geometry>
-        <box size="${camera_link} ${camera_link} ${camera_link}"/>
-            </geometry>
-            <material name="red"/>
+                <box size="${camera_link} ${camera_link} ${camera_link}"/>
+                <!-- <mesh filename="file://$(find bioloid_typea_description)/assets/cad/camera.dae" scale="0.01 0.01 0.01"/> -->
+            </geometry>
         </visual>
         <inertial>

Commit message: Teledyne 3D added to bioloid Xacro file.

File: src/bioloid_typea_description/gazebo.xacro (robot description, xacro)
@@ -29,11 +29,13 @@
     <gazebo reference="camera_link">
         <sensor type="camera" name="camera">
-            <update_rate>30.0</update_rate>
+            <update_rate>22.7</update_rate>
             <camera name="head">
                 <horizontal_fov>1.3962634</horizontal_fov>
                 <image>
-                  <width>800</width>
-                  <height>800</height>
-                  <format>R8G8B8</format>
+                    <!--<width>2592</width>
+                    <height>2048</height>-->
+                    <width>480</width>
+                    <height>380</height>
+                    <format>R8G8B8</format>
                 </image>
                 <clip>

File: src/bioloid_typea_description/typea.xacro (robot description, xacro)
@@ -35,5 +35,5 @@
     <xacro:include filename="$(find bioloid_typea_description)/std_parts.xacro"/>
      <xacro:property name="camera_link" value="0.01" />
-     <xacro:property name="height_camera" value="0.157"/>
+     <xacro:property name="height_camera" value="0.167"/>
      <xacro:property name="axel_offset" value="0.05"/>
     <!-- Camera -->
@@ -52,12 +52,12 @@
         </collision>
         <visual>
-            <origin xyz="0 0 0" rpy="0 0 0"/>
-            <geometry>
-                <box size="${camera_link} ${camera_link} ${camera_link}"/>
-                <!-- <mesh filename="file://$(find bioloid_typea_description)/assets/cad/camera.dae" scale="0.01 0.01 0.01"/> -->
-            </geometry>
-        </visual>
-        <inertial>
-            <mass value="1e-5" />
+            <origin xyz="0 0 0" rpy="0 0 -1.5707"/>
+            <geometry>
+               <!-- <box size="${camera_link} ${camera_link} ${camera_link}"/> -->
+                <mesh filename="file://$(find bioloid_typea_description)/assets/cad/teledyne.dae"/>
+            </geometry>
+        </visual>
+        <inertial>
+            <mass value="0.046" />
             <origin xyz="0 0 0" rpy="0 0 0"/>
             <inertia ixx="1e-6" ixy="0" ixz="0" iyy="1e-6" iyz="0" izz="1e-6" />
