Commit message: Updating Move To and Xacro Files.

File: src/bioloid_typea_description/typea.urdf (robot description, URDF)
Before this commit: robot typea, 25 links, 24 joints
Links:
- removed link l_ankle_lateral_link
- removed link l_ankle_swing_link
- removed link l_foot_link
- removed link l_hip_lateral_link
- removed link l_hip_twist_link
- removed link l_lower_leg_link
- removed link l_upper_leg_link
- removed link r_ankle_lateral_link
- removed link r_ankle_swing_link
- removed link r_foot_link
- removed link r_hip_lateral_link
- removed link r_hip_twist_link
- removed link r_lower_leg_link
- removed link r_upper_leg_link
- removed link torso_link
- added link camera_link, mass 0.046; collision box size=${camera_link} ${camera_link} ${camera_link}; visual mesh filename=file://$(find bioloid_typea_description)/assets/cad/teledyn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
- link l_hand_link: mass 0.0303003163 -> None; geometry collision box size=0.0131 0.0265 0.044; collision box size=0.0575 0.0175 0.035
- link l_lower_arm_link: mass 0.3822870734 -> None; geometry collision box size=0.058 0.033 0.044
- link l_shoulder_swing_link: mass 0.0595945816 -> None; geometry collision box size=0.052 0.039 0.036
- link l_upper_arm_link: mass 0.3822870734 -> None; geometry collision box size=0.047 0.033 0.052; collision box size=0.054 0.033 0.044
- link r_hand_link: mass 0.0303003163 -> None; geometry collision box size=0.0131 0.0265 0.044; collision box size=0.0575 0.0175 0.035
- link r_lower_arm_link: mass 0.3833833954 -> None; geometry collision box size=0.058 0.033 0.044
- link r_shoulder_swing_link: mass 0.0595945816 -> None; geometry collision box size=0.052 0.039 0.036
- link r_upper_arm_link: mass 0.3822870734 -> None; geometry collision box size=0.047 0.033 0.052; collision box size=0.054 0.033 0.044
Joints:
- removed joint l_ankle_lateral_joint
- removed joint l_ankle_swing_joint
- removed joint l_elbow_joint
- removed joint l_foot_joint
- removed joint l_hand_joint
- removed joint l_hip_lateral_joint
- removed joint l_hip_swing_joint
- removed joint l_hip_twist_joint
- removed joint l_knee_joint
- removed joint l_shoulder_lateral_joint
- removed joint l_shoulder_swing_joint
- removed joint r_ankle_lateral_joint
- removed joint r_ankle_swing_joint
- removed joint r_elbow_joint
- removed joint r_foot_joint
- removed joint r_hand_joint
- removed joint r_hip_lateral_joint
- removed joint r_hip_swing_joint
- removed joint r_hip_twist_joint
- removed joint r_knee_joint
- removed joint r_shoulder_lateral_joint
- removed joint r_shoulder_swing_joint
- added joint camera_joint: type fixed, parent base_link, child camera_link, origin xyz=${camera_link} 0 ${height_camera - axel_offset*2} rpy=0 0 0, axis 0 1 0

File: src/bioloid_typea_description/typea.xacro (robot description, xacro)
@@ -48,5 +48,5 @@
             <origin xyz="0 0 0" rpy="0 0 0"/>
             <geometry>
-        <box size="${camera_link} ${camera_link} ${camera_link}"/>
+                <box size="${camera_link} ${camera_link} ${camera_link}"/>
             </geometry>
         </collision>
